Commit message: normalize joint orientation

File: config/we_r2_arm.urdf.xacro (robot description, xacro)
@@ -6,6 +6,5 @@
     <origin rpy="0 0 0" xyz="0 0 0"/>
     <geometry>
-      <mesh filename="package://we_r2_moveit_config/config/bin_stl/base_link_m-binary.stl"/>-->
-      <!--<cylinder length="0.42" radius="0.07"/>-->
+      <mesh filename="package://we_r2_moveit_config/config/bin_stl/base_link_m-binary.stl"/>
     </geometry>
     <material name="silver">
@@ -16,21 +15,82 @@
     <origin rpy="0 0 0" xyz="0 0 0"/>
     <geometry>
-      <xacro:if value="${simple_collision}">
-        <cylinder length="0.42" radius="0.07"/>
-      </xacro:if>
-      <xacro:unless value="${simple_collision}">
-        <mesh filename="package://we_r2_moveit_config/config/bin_stl/base_link_m-binary.stl"/>
-      </xacro:unless>
-     </geometry>
+      <mesh filename="package://we_r2_moveit_config/config/bin_stl/base_link_m-binary.stl"/>
+    </geometry>
+  </collision>
+</link>
+<link name="Forearm__1">
+  <inertial>
+    <origin rpy="0 0 0" xyz="-0.014792 -0.00013599999999999723 0.101354"/>
+    <mass value="0.670217"/>
+    <inertia ixx="0.004244" ixy="0.0" ixz="0.007572" iyy="0.004259" iyz="-0.007549" izz="0.000301"/>
+  </inertial>
+  <visual>
+    <origin rpy="0 0 0" xyz="0.035775 0.074529 -0.366958"/>
+    <geometry>
+      <mesh filename="package://we_r2_moveit_config/config/bin_stl/Forearm__1_m-binary.stl"/>
+    </geometry>
+    <material name="silver">
+      <color rgba="1 0 0 1"/>
+    </material>
+  </visual>
+  <collision>
+    <origin rpy="0 0 0" xyz="0.035775 0.074529 -0.366958"/>
+    <geometry>
+      <mesh filename="package://we_r2_moveit_config/config/bin_stl/Forearm__1_m-binary.stl"/>
+    </geometry>
+  </collision>
+</link>
+<link name="wrist_1__1">
+  <inertial>
+    <origin rpy="0 0 0" xyz="0.025382 -1.000000000001e-06 0.0072510000000000074"/>
+    <mass value="0.282343"/>
+    <inertia ixx="0.000154" ixy="0.0" ixz="0.011825" iyy="0.000162" iyz="-0.011831" izz="0.000133"/>
+  </inertial>
+  <visual>
+    <origin rpy="0 0 0" xyz="0.024453 0.074942 -0.544758"/>
+    <geometry>
+      <mesh filename="package://we_r2_moveit_config/config/bin_stl/wrist_1__1_m-binary.stl"/>
+    </geometry>
+    <material name="silver">
+      <color rgba="1 0 0 1"/>
+    </material>
+  </visual>
+  <collision>
+    <origin rpy="0 0 0" xyz="0.024453 0.074942 -0.544758"/>
+    <geometry>
+      <mesh filename="package://we_r2_moveit_config/config/bin_stl/wrist_1__1_m-binary.stl"/>
+    </geometry>
+  </collision>
+</link>
+<link name="upper_arm__1">
+  <inertial>
+    <origin rpy="0 0 0" xyz="-0.015592 -6.1000000000005494e-05 0.20106100000000002"/>
+    <mass value="0.465826"/>
+    <inertia ixx="0.000327" ixy="0.0" ixz="0.012132" iyy="0.000496" iyz="-0.012106" izz="0.000474"/>
+  </inertial>
+  <visual>
+    <origin rpy="0 0 0" xyz="-0.012324 0.074585 -0.163809"/>
+    <geometry>
+      <mesh filename="package://we_r2_moveit_config/config/bin_stl/upper_arm__1_m-binary.stl"/>
+    </geometry>
+    <material name="silver">
+      <color rgba="1 0 0 1"/>
+    </material>
+  </visual>
+  <collision>
+    <origin rpy="0 0 0" xyz="-0.012324 0.074585 -0.163809"/>
+    <geometry>
+      <mesh filename="package://we_r2_moveit_config/config/bin_stl/upper_arm__1_m-binary.stl"/>
+    </geometry>
   </collision>
 </link>
 <link name="shoulder__1">
   <inertial>
-    <origin rpy="0 0 0" xyz="0.019128000000000003 0.0008300000000000002 0.042733999999999994"/>
+    <origin rpy="0 0 0" xyz="-0.019159 8.900000000000574e-05 0.04272799999999999"/>
     <mass value="1.493039"/>
-    <inertia ixx="0.002393" ixy="-1.2e-05" ixz="0.003808" iyy="0.002653" iyz="-0.003962" izz="0.001979"/>
-  </inertial>
-  <visual>
-    <origin rpy="0 0 0" xyz="-0.000148 -0.00137 -0.106993"/>
+    <inertia ixx="0.002392" ixy="2e-06" ixz="0.012495" iyy="0.002653" iyz="-0.012347" izz="0.001979"/>
+  </inertial>
+  <visual>
+    <origin rpy="0 0 0" xyz="-0.000666 0.07459 -0.106659"/>
     <geometry>
       <mesh filename="package://we_r2_moveit_config/config/bin_stl/shoulder__1_m-binary.stl"/>
@@ -41,5 +101,5 @@
   </visual>
   <collision>
-    <origin rpy="0 0 0" xyz="-0.000148 -0.00137 -0.106993"/>
+    <origin rpy="0 0 0" xyz="-0.000666 0.07459 -0.106659"/>
     <geometry>
       <mesh filename="package://we_r2_moveit_config/config/bin_stl/shoulder__1_m-binary.stl"/>
@@ -47,12 +107,34 @@
   </collision>
 </link>
+<link name="wrist_2__1">
+  <inertial>
+    <origin rpy="0 0 0" xyz="-3.399999999999974e-05 0.007306999999999994 0.025361000000000078"/>
+    <mass value="0.282365"/>
+    <inertia ixx="0.000162" ixy="-0.0" ixz="0.011849" iyy="0.000133" iyz="-0.011855" izz="0.000155"/>
+  </inertial>
+  <visual>
+    <origin rpy="0 0 0" xyz="-0.002217 0.074916 -0.576213"/>
+    <geometry>
+      <mesh filename="package://we_r2_moveit_config/config/bin_stl/wrist_2__1_m-binary.stl"/>
+    </geometry>
+    <material name="silver">
+      <color rgba="1 0 0 1"/>
+    </material>
+  </visual>
+  <collision>
+    <origin rpy="0 0 0" xyz="-0.002217 0.074916 -0.576213"/>
+    <geometry>
+      <mesh filename="package://we_r2_moveit_config/config/bin_stl/wrist_2__1_m-binary.stl"/>
+    </geometry>
+  </collision>
+</link>
 <link name="end_effector_link__1">
   <inertial>
-    <origin rpy="0 0 0" xyz="-0.003476 -0.0016250000000000153 -0.006948999999999997"/>
+    <origin rpy="0 0 0" xyz="-3.800000000000027e-05 0.007937999999999994 -1.8000000000073513e-05"/>
     <mass value="0.0358"/>
-    <inertia ixx="5e-06" ixy="1e-06" ixz="0.000677" iyy="1.2e-05" iyz="-0.000674" izz="1e-05"/>
-  </inertial>
-  <visual>
-    <origin rpy="0 0 0" xyz="0.003959 0.223317 -0.09394"/>
+    <inertia ixx="3e-06" ixy="-0.0" ixz="0.000809" iyy="1.2e-05" iyz="-0.000809" izz="1.2e-05"/>
+  </inertial>
+  <visual>
+    <origin rpy="0 0 0" xyz="-0.002069 0.043403 -0.602813"/>
     <geometry>
       <mesh filename="package://we_r2_moveit_config/config/bin_stl/end_effector_link__1_m-binary.stl"/>
@@ -63,5 +145,5 @@
   </visual>
   <collision>
-    <origin rpy="0 0 0" xyz="0.003959 0.223317 -0.09394"/>
+    <origin rpy="0 0 0" xyz="-0.002069 0.043403 -0.602813"/>
     <geometry>
       <mesh filename="package://we_r2_moveit_config/config/bin_stl/end_effector_link__1_m-binary.stl"/>
@@ -69,97 +151,89 @@
   </collision>
 </link>
-<link name="upper_arm__1">
-  <inertial>
-    <origin rpy="0 0 0" xyz="0.023742 -0.158727 0.122109"/>
-    <mass value="0.465826"/>
-    <inertia ixx="0.000325" ixy="1.2e-05" ixz="0.022719" iyy="0.000484" iyz="-0.022725" izz="0.000488"/>
-  </inertial>
-  <visual>
-    <origin rpy="0 0 0" xyz="0.011507 -0.000645 -0.164119"/>
-    <geometry>
-      <mesh filename="package://we_r2_moveit_config/config/bin_stl/upper_arm__1_m-binary.stl"/>
-    </geometry>
-    <material name="silver">
-      <color rgba="1 0 0 1"/>
-    </material>
-  </visual>
-  <collision>
-    <origin rpy="0 0 0" xyz="0.011507 -0.000645 -0.164119"/>
-    <geometry>
-      <mesh filename="package://we_r2_moveit_config/config/bin_stl/upper_arm__1_m-binary.stl"/>
-    </geometry>
-  </collision>
-</link>
-<link name="Forearm__1">
-  <inertial>
-    <origin rpy="0 0 0" xyz="0.014801000000000002 0.0008319999999999994 -0.101349"/>
-    <mass value="0.670217"/>
-    <inertia ixx="0.004243" ixy="-1e-06" ixz="0.027051" iyy="0.004259" iyz="-0.027034" izz="0.000301"/>
-  </inertial>
-  <visual>
-    <origin rpy="0 0 0" xyz="-0.044786 0.158107 -0.287456"/>
-    <geometry>
-      <mesh filename="package://we_r2_moveit_config/config/bin_stl/Forearm__1_m-binary.stl"/>
-    </geometry>
-    <material name="silver">
-      <color rgba="1 0 0 1"/>
-    </material>
-  </visual>
-  <collision>
-    <origin rpy="0 0 0" xyz="-0.044786 0.158107 -0.287456"/>
-    <geometry>
-      <mesh filename="package://we_r2_moveit_config/config/bin_stl/Forearm__1_m-binary.stl"/>
-    </geometry>
-  </collision>
-</link>
-<link name="wrist_1__1">
-  <inertial>
-    <origin rpy="0 0 0" xyz="-0.024984000000000003 -0.00839999999999999 0.0014440000000000008"/>
-    <mass value="0.282343"/>
-    <inertia ixx="0.000155" ixy="-5e-06" ixz="0.005515" iyy="0.000133" iyz="-0.005508" izz="0.000161"/>
-  </inertial>
-  <visual>
-    <origin rpy="0 0 0" xyz="-0.033535 0.158674 -0.109652"/>
-    <geometry>
-      <mesh filename="package://we_r2_moveit_config/config/bin_stl/wrist_1__1_m-binary.stl"/>
-    </geometry>
-    <material name="silver">
-      <color rgba="1 0 0 1"/>
-    </material>
-  </visual>
-  <collision>
-    <origin rpy="0 0 0" xyz="-0.033535 0.158674 -0.109652"/>
-    <geometry>
-        <mesh filename="package://we_r2_moveit_config/config/bin_stl/wrist_1__1_m-binary.stl"/>
-    </geometry>
-  </collision>
-</link>
-<link name="wrist_2__1">
-  <inertial>
-    <origin rpy="0 0 0" xyz="-0.0019010000000000008 -0.026297999999999988 -0.0011819999999999886"/>
-    <mass value="0.282365"/>
-    <inertia ixx="0.000157" ixy="-5e-06" ixz="0.007246" iyy="0.000151" iyz="-0.007265" izz="0.000142"/>
-  </inertial>
-  <visual>
-    <origin rpy="0 0 0" xyz="-0.008481 0.190801 -0.116045"/>
-    <geometry>
-      <mesh filename="package://we_r2_moveit_config/config/bin_stl/wrist_2__1_m-binary.stl"/>
-    </geometry>
-    <material name="silver">
-      <color rgba="1 0 0 1"/>
-    </material>
-  </visual>
-  <collision>
-    <origin rpy="0 0 0" xyz="-0.008481 0.190801 -0.116045"/>
-    <geometry>
-      <mesh filename="package://we_r2_moveit_config/config/bin_stl/wrist_2__1_m-binary.stl"/>
-    </geometry>
-  </collision>
-</link>
+<joint name="joint2" type="continuous">
+  <origin rpy="0 0 0" xyz="-0.048099 5.6e-05 0.203149"/>
+  <parent link="upper_arm__1"/>
+  <child link="Forearm__1"/>
+  <axis xyz="-0.01 1.7e-05 0.0"/>
+</joint>
+<transmission name="joint2_tran">
+  <type>transmission_interface/SimpleTransmission</type>
+  <joint name="joint2">
+    <hardwareInterface>PositionJointInterface</hardwareInterface>
+  </joint>
+  <actuator name="joint2_actr">
+    <hardwareInterface>PositionJointInterface</hardwareInterface>
+    <mechanicalReduction>1</mechanicalReduction>
+  </actuator>
+</transmission>
+<joint name="joint3" type="continuous">
+  <origin rpy="0 0 0" xyz="0.011322 -0.000413 0.1778"/>
+  <parent link="Forearm__1"/>
+  <child link="wrist_1__1"/>
+  <axis xyz="0.01 -1.7e-05 -0.0"/>
+</joint>
+<transmission name="joint3_tran">
+  <type>transmission_interface/SimpleTransmission</type>
+  <joint name="joint3">
+    <hardwareInterface>PositionJointInterface</hardwareInterface>
+  </joint>
+  <actuator name="joint3_actr">
+    <hardwareInterface>PositionJointInterface</hardwareInterface>
+    <mechanicalReduction>1</mechanicalReduction>
+  </actuator>
+</transmission>
+<joint name="joint1" type="continuous">
+  <origin rpy="0 0 0" xyz="0.011658 5e-06 0.05715"/>
+  <parent link="shoulder__1"/>
+  <child link="upper_arm__1"/>
+  <axis xyz="0.01 -1.7e-05 0.0"/>
+</joint>
+<transmission name="joint1_tran">
+  <type>transmission_interface/SimpleTransmission</type>
+  <joint name="joint1">
+    <hardwareInterface>PositionJointInterface</hardwareInterface>
+  </joint>
+  <actuator name="joint1_actr">
+    <hardwareInterface>PositionJointInterface</hardwareInterface>
+    <mechanicalReduction>1</mechanicalReduction>
+  </actuator>
+</transmission>
+<joint name="joint0" type="continuous">
+  <origin rpy="0 0 0" xyz="0.000666 -0.07459 0.106659"/>
+  <parent link="base_link"/>
+  <child link="shoulder__1"/>
+  <axis xyz="0.0 0.0 0.01"/>
+</joint>
+<transmission name="joint0_tran">
+  <type>transmission_interface/SimpleTransmission</type>
+  <joint name="joint0">
+    <hardwareInterface>PositionJointInterface</hardwareInterface>
+  </joint>
+  <actuator name="joint0_actr">
+    <hardwareInterface>PositionJointInterface</hardwareInterface>
+    <mechanicalReduction>1</mechanicalReduction>
+  </actuator>
+</transmission>
+<joint name="joint4" type="continuous">
+  <origin rpy="0 0 0" xyz="0.02667 2.6e-05 0.031455"/>
+  <parent link="wrist_1__1"/>
+  <child link="wrist_2__1"/>
+  <axis xyz="0.0 2.2e-05 0.01"/>
+</joint>
+<transmission name="joint4_tran">
+  <type>transmission_interface/SimpleTransmission</type>
+  <joint name="joint4">
+    <hardwareInterface>PositionJointInterface</hardwareInterface>
+  </joint>
+  <actuator name="joint4_actr">
+    <hardwareInterface>PositionJointInterface</hardwareInterface>
+    <mechanicalReduction>1</mechanicalReduction>
+  </actuator>
+</transmission>
 <joint name="joint5" type="continuous">
-  <origin rpy="0 0 0" xyz="-0.01244 -0.032516 -0.022105"/>
+  <origin rpy="0 0 0" xyz="-0.000148 0.031513 0.0266"/>
   <parent link="wrist_2__1"/>
   <child link="end_effector_link__1"/>
-  <axis xyz="-0.004381 -0.002047 -0.008753"/>
+  <axis xyz="-4.7e-05 0.01 -2.2e-05"/>
 </joint>
 <transmission name="joint5_tran">
@@ -169,84 +243,4 @@
   </joint>
   <actuator name="joint5_actr">
-    <hardwareInterface>PositionJointInterface</hardwareInterface>
-    <mechanicalReduction>1</mechanicalReduction>
-  </actuator>
-</transmission>
-<joint name="joint1" type="continuous">
-  <origin rpy="0 0 0" xyz="-0.011655 -0.000725 0.057126"/>
-  <parent link="shoulder__1"/>
-  <child link="upper_arm__1"/>
-  <axis xyz="-0.009987 -0.000514 -3e-06"/>
-</joint>
-<transmission name="joint1_tran">
-  <type>transmission_interface/SimpleTransmission</type>
-  <joint name="joint1">
-    <hardwareInterface>PositionJointInterface</hardwareInterface>
-  </joint>
-  <actuator name="joint1_actr">
-    <hardwareInterface>PositionJointInterface</hardwareInterface>
-    <mechanicalReduction>1</mechanicalReduction>
-  </actuator>
-</transmission>
-<joint name="joint2" type="continuous">
-  <origin rpy="0 0 0" xyz="0.056293 -0.158752 0.123337"/>
-  <parent link="upper_arm__1"/>
-  <child link="Forearm__1"/>
-  <axis xyz="0.009987 0.000514 3e-06"/>
-</joint>
-<transmission name="joint2_tran">
-  <type>transmission_interface/SimpleTransmission</type>
-  <joint name="joint2">
-    <hardwareInterface>PositionJointInterface</hardwareInterface>
-  </joint>
-  <actuator name="joint2_actr">
-    <hardwareInterface>PositionJointInterface</hardwareInterface>
-    <mechanicalReduction>1</mechanicalReduction>
-  </actuator>
-</transmission>
-<joint name="joint0" type="continuous">
-  <origin rpy="0 0 0" xyz="0.000148 0.00137 0.106993"/>
-  <parent link="base_link"/>
-  <child link="shoulder__1"/>
-  <axis xyz="-2e-06 -2.3e-05 0.01"/>
-</joint>
-<transmission name="joint0_tran">
-  <type>transmission_interface/SimpleTransmission</type>
-  <joint name="joint0">
-    <hardwareInterface>PositionJointInterface</hardwareInterface>
-  </joint>
-  <actuator name="joint0_actr">
-    <hardwareInterface>PositionJointInterface</hardwareInterface>
-    <mechanicalReduction>1</mechanicalReduction>
-  </actuator>
-</transmission>
-<joint name="joint3" type="continuous">
-  <origin rpy="0 0 0" xyz="-0.011251 -0.000567 -0.177804"/>
-  <parent link="Forearm__1"/>
-  <child link="wrist_1__1"/>
-  <axis xyz="-0.009987 -0.000514 -3e-06"/>
-</joint>
-<transmission name="joint3_tran">
-  <type>transmission_interface/SimpleTransmission</type>
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
Commit message: default joint limits

File: config/we_r2_arm.urdf.xacro (robot description, xacro)
@@ -15,5 +15,10 @@
     <origin rpy="0 0 0" xyz="0 0 0"/>
     <geometry>
-      <mesh filename="package://we_r2_moveit_config/config/bin_stl/base_link_m-binary.stl"/>
+      <xacro:if value="${simple_collision}">
+        <cylinder length="0.42" radius="0.07"/>
+      </xacro:if>
+      <xacro:unless value="${simple_collision}">
+        <mesh filename="package://we_r2_moveit_config/config/bin_stl/base_link_m-binary.stl"/>
+      </xacro:unless>
     </geometry>
   </collision>
@@ -151,9 +156,10 @@
   </collision>
 </link>
-<joint name="joint2" type="continuous">
+<joint name="joint2" type="revolute">
   <origin rpy="0 0 0" xyz="-0.048099 5.6e-05 0.203149"/>
   <parent link="upper_arm__1"/>
   <child link="Forearm__1"/>
   <axis xyz="-0.01 1.7e-05 0.0"/>
+  <limit effort="100" velocity="1.0" lower="-6.5" upper="6.5" />
 </joint>
 <transmission name="joint2_tran">
@@ -167,9 +173,10 @@
   </actuator>
 </transmission>
-<joint name="joint3" type="continuous">
+<joint name="joint3" type="revolute">
   <origin rpy="0 0 0" xyz="0.011322 -0.000413 0.1778"/>
   <parent link="Forearm__1"/>
   <child link="wrist_1__1"/>
   <axis xyz="0.01 -1.7e-05 -0.0"/>
+  <limit effort="100" velocity="1.0" lower="-6.5" upper="6.5" />
 </joint>
 <transmission name="joint3_tran">
@@ -183,9 +190,10 @@
   </actuator>
 </transmission>
-<joint name="joint1" type="continuous">
+<joint name="joint1" type="revolute">
   <origin rpy="0 0 0" xyz="0.011658 5e-06 0.05715"/>
   <parent link="shoulder__1"/>
   <child link="upper_arm__1"/>
   <axis xyz="0.01 -1.7e-05 0.0"/>
+  <limit effort="100" velocity="1.0" lower="-6.5" upper="6.5" />
 </joint>
 <transmission name="joint1_tran">
@@ -199,9 +207,10 @@
   </actuator>
 </transmission>
-<joint name="joint0" type="continuous">
+<joint name="joint0" type="revolute">
   <origin rpy="0 0 0" xyz="0.000666 -0.07459 0.106659"/>
   <parent link="base_link"/>
   <child link="shoulder__1"/>
   <axis xyz="0.0 0.0 0.01"/>
+  <limit effort="100" velocity="1.0" lower="-6.5" upper="6.5" />
 </joint>
 <transmission name="joint0_tran">
@@ -215,9 +224,10 @@
   </actuator>
 </transmission>
-<joint name="joint4" type="continuous">
+<joint name="joint4" type="revolute">
   <origin rpy="0 0 0" xyz="0.02667 2.6e-05 0.031455"/>
   <parent link="wrist_1__1"/>
   <child link="wrist_2__1"/>
   <axis xyz="0.0 2.2e-05 0.01"/>
+  <limit effort="100" velocity="1.0" lower="-6.5" upper="6.5" />
 </joint>
 <transmission name="joint4_tran">
@@ -231,9 +241,10 @@
   </actuator>
 </transmission>
-<joint name="joint5" type="continuous">
+<joint name="joint5" type="revolute">
   <origin rpy="0 0 0" xyz="-0.000148 0.031513 0.0266"/>
   <parent link="wrist_2__1"/>
   <child link="end_effector_link__1"/>
   <axis xyz="-4.7e-05 0.01 -2.2e-05"/>
+  <limit effort="100" velocity="1.0" lower="-6.5" upper="6.5" />
 </joint>
 <transmission name="joint5_tran">

Commit message: fix joint

File: config/we_r2_arm.urdf.xacro (robot description, xacro)
@@ -207,10 +207,9 @@
   </actuator>
 </transmission>
-<joint name="joint0" type="revolute">
+<joint name="joint0" type="continuous">
   <origin rpy="0 0 0" xyz="0.000666 -0.07459 0.106659"/>
   <parent link="base_link"/>
   <child link="shoulder__1"/>
   <axis xyz="0.0 0.0 0.01"/>
-  <limit effort="100" velocity="1.0" lower="-6.5" upper="6.5" />
 </joint>
 <transmission name="joint0_tran">

Commit message: simple joint position execution

File: config/we_r2_arm.urdf.xacro (robot description, xacro)
@@ -156,10 +156,10 @@
   </collision>
 </link>
-<joint name="joint2" type="revolute">
+<joint name="joint2" type="continuous">
   <origin rpy="0 0 0" xyz="-0.048099 5.6e-05 0.203149"/>
   <parent link="upper_arm__1"/>
   <child link="Forearm__1"/>
   <axis xyz="-0.01 1.7e-05 0.0"/>
-  <limit effort="100" velocity="1.0" lower="-6.5" upper="6.5" />
+  <limit effort="100" velocity="0.1"/>
 </joint>
 <transmission name="joint2_tran">
@@ -173,10 +173,10 @@
   </actuator>
 </transmission>
-<joint name="joint3" type="revolute">
+<joint name="joint3" type="continuous">
   <origin rpy="0 0 0" xyz="0.011322 -0.000413 0.1778"/>
   <parent link="Forearm__1"/>
   <child link="wrist_1__1"/>
   <axis xyz="0.01 -1.7e-05 -0.0"/>
-  <limit effort="100" velocity="1.0" lower="-6.5" upper="6.5" />
+  <limit effort="100" velocity="0.1"/>
 </joint>
 <transmission name="joint3_tran">
@@ -190,10 +190,10 @@
   </actuator>
 </transmission>
-<joint name="joint1" type="revolute">
+<joint name="joint1" type="continuous">
   <origin rpy="0 0 0" xyz="0.011658 5e-06 0.05715"/>
   <parent link="shoulder__1"/>
   <child link="upper_arm__1"/>
   <axis xyz="0.01 -1.7e-05 0.0"/>
-  <limit effort="100" velocity="1.0" lower="-6.5" upper="6.5" />
+  <limit effort="100" velocity="0.1"/>
 </joint>
 <transmission name="joint1_tran">
@@ -212,4 +212,5 @@
   <child link="shoulder__1"/>
   <axis xyz="0.0 0.0 0.01"/>
+  <limit effort="100" velocity="0.1"/>
 </joint>
 <transmission name="joint0_tran">
@@ -223,10 +224,10 @@
   </actuator>
 </transmission>
-<joint name="joint4" type="revolute">
+<joint name="joint4" type="continuous">
   <origin rpy="0 0 0" xyz="0.02667 2.6e-05 0.031455"/>
   <parent link="wrist_1__1"/>
   <child link="wrist_2__1"/>
   <axis xyz="0.0 2.2e-05 0.01"/>
-  <limit effort="100" velocity="1.0" lower="-6.5" upper="6.5" />
+  <limit effort="100" velocity="0.1"/>
 </joint>
 <transmission name="joint4_tran">
@@ -240,10 +241,10 @@
   </actuator>
 </transmission>
-<joint name="joint5" type="revolute">
+<joint name="joint5" type="continuous">
   <origin rpy="0 0 0" xyz="-0.000148 0.031513 0.0266"/>
   <parent link="wrist_2__1"/>
   <child link="end_effector_link__1"/>
   <axis xyz="-4.7e-05 0.01 -2.2e-05"/>
-  <limit effort="100" velocity="1.0" lower="-6.5" upper="6.5" />
+  <limit effort="100" velocity="0.1"/>
 </joint>
 <transmission name="joint5_tran">

Commit message: simple joint position execution

File: config/we_r2_arm.urdf.xacro (robot description, xacro)
@@ -161,5 +161,5 @@
   <child link="Forearm__1"/>
   <axis xyz="-0.01 1.7e-05 0.0"/>
-  <limit effort="100" velocity="0.1"/>
+  <limit effort="100" velocity="0.5"/>
 </joint>
 <transmission name="joint2_tran">
@@ -178,5 +178,5 @@
   <child link="wrist_1__1"/>
   <axis xyz="0.01 -1.7e-05 -0.0"/>
-  <limit effort="100" velocity="0.1"/>
+  <limit effort="100" velocity="0.5"/>
 </joint>
 <transmission name="joint3_tran">
@@ -195,5 +195,5 @@
   <child link="upper_arm__1"/>
   <axis xyz="0.01 -1.7e-05 0.0"/>
-  <limit effort="100" velocity="0.1"/>
+  <limit effort="100" velocity="0.5"/>
 </joint>
 <transmission name="joint1_tran">
@@ -212,5 +212,5 @@
   <child link="shoulder__1"/>
   <axis xyz="0.0 0.0 0.01"/>
-  <limit effort="100" velocity="0.1"/>
+  <limit effort="100" velocity="0.5"/>
 </joint>
 <transmission name="joint0_tran">
@@ -229,5 +229,5 @@
   <child link="wrist_2__1"/>
   <axis xyz="0.0 2.2e-05 0.01"/>
-  <limit effort="100" velocity="0.1"/>
+  <limit effort="100" velocity="0.5"/>
 </joint>
 <transmission name="joint4_tran">
@@ -246,5 +246,5 @@
   <child link="end_effector_link__1"/>
   <axis xyz="-4.7e-05 0.01 -2.2e-05"/>
-  <limit effort="100" velocity="0.1"/>
+  <limit effort="100" velocity="0.5"/>
 </joint>
 <transmission name="joint5_tran">
